Commit message: cmpIMU
conver Quanternion to euler angles

File: install/balegce/share/balegce/robot/visual/manipulator.xacro (robot description, xacro)
@@ -140,5 +140,6 @@
         </collision>
     </xacro:macro>
-    <xacro:macro name="base" params="">
+    <!-- <xacro:macro name="base" params=""> -->
+    <xacro:macro name="base_offset" params="">
         <joint name="base" type="fixed">
             <parent link="base"/>
@@ -223,5 +224,6 @@
             <xacro:propeller_collision />
         </link>
-        <xacro:base/>
+        <!-- <xacro:base/> -->
+        <xacro:base_offset/>
         <xacro:joint_body/>
         <xacro:joint_wheel/>

File: install/balegce_gazebo/share/balegce_gazebo/robot/balegce.gazebo.xacro (robot description, xacro)
@@ -11,5 +11,10 @@
     <xacro:include filename="$(find ${description_pkg})/robot/visual/manipulator.xacro"/>
     <xacro:include filename="$(find ${description_package})/robot/visual/sensor.xacro"/>
+    <!-- <link name="world"/> -->
     <xacro:balegce/>
+    <!-- <joint name="offset" type="floating">
+        <parent link="world"/>
+        <child link="base"/>
+    </joint> -->
     <xacro:sensor_link/>
     <xacro:sensor_plugins/>
